File: mp3b/mp3b.kicad_pcb (KiCad board)
At the start: 2 copper layers, 37.2 x 40.1 mm, 35 parts, among them J1 USB_microB_2040002-1, J2 Arduino_ICSP, J3 Conn_01x15_Male, J4 Conn_01x15_Male, U1 FT232RL, U2 MCP1702T-5002E_CB, U3 TPS2113ADRBR, U4 ATMEGA328PB-ANR, Y1 16MHz

Commit message: Update mp3b.kicad_pcb
Routing:
- net Net-(C7-Pad1): track 43.8 -> 55.0 mm
- net +5V: track 129.8 -> 124.5 mm, vias 11 -> 9
- net GND: track 192.0 -> 196.8 mm, vias 19 -> 22
- net /A0: track 57.5 -> 55.6 mm
- net /D11: track 73.5 -> 72.1 mm
- net /A7: track 37.1 -> 36.2 mm
- net Net-(D2-Pad1): track 3.36 -> 2.79 mm
- net /AREF: track 48.0 -> 47.4 mm, vias 2 -> 1
- net /D12: track 59.2 -> 58.7 mm, vias 3 -> 1
